File: HW/light/light.sch (KiCad schematic (older format))
At the start: 48 parts, among them P1 Battery, P2 USB_A, P3 ISP, Q1 BSS138, SW1 ON, SW2 OFF, U1 MCP73831, U10 APA102, U11 APA102, U12 APA102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

Commit message: Add documents
Parts:
- removed C10, C11, C12, C13, C14, C3, C5, C6, C7, C8, C9: 1uF, Capacitors_SMD:C_0603_HandSoldering, symbol C_Small
- removed D2: Charge, LEDs:LED_0603, symbol LED_Small
- removed P2: USB_A, Connect:USB_Mini-B, symbol USB_OTG
- removed P3: ISP, Pin_Headers:Pin_Header_Straight_1x06, symbol CONN_01X06
- removed Q1: BSS138, TO_SOT_Packages_SMD:SOT-23_Handsoldering, symbol BSS138
- removed R10, R9: 4,7K, Resistors_SMD:R_0603_HandSoldering, symbol R_Small
- removed R11: 470, Resistors_SMD:R_0603_HandSoldering, symbol R_Small
- removed R12: 2K, Resistors_SMD:R_0603_HandSoldering, symbol R_Small
- removed R2: 100, Resistors_SMD:R_0603_HandSoldering, symbol R_Small
- removed R3: 100K, Resistors_SMD:R_0603_HandSoldering, symbol R_Small
- removed R4: 1M, Resistors_SMD:R_0603_HandSoldering, symbol R_Small
- removed R5, R6: 1K, Resistors_SMD:R_0603_HandSoldering, symbol R_Small
- removed SW1: ON, Buttons_Switches_ThroughHole:SW_Tactile_SPST_Angled, symbol SW_PUSH
- removed SW2: OFF, Buttons_Switches_ThroughHole:SW_Tactile_SPST_Angled, symbol SW_PUSH
- removed U1: MCP73831, suf_sot:SOT-23-5_Handsoldering, symbol MCP73831
- removed U10, U11, U12, U13, U4, U5, U6, U7, U8, U9: APA102, LEDs:LED_WS2812-PLCC6, symbol APA102
- added C? (x25): 1uF, Capacitors_SMD:C_0603_HandSoldering, symbol C_Small
- added CON?: AVR-ISP-6, AVR-ISP-6, symbol AVR-ISP-6
- added R?: 470, Resistors_SMD:R_0603_HandSoldering, symbol R_Small
- added U?: LP2980, symbol LP2980
- added U? (x24): SK6812_MINI, suf_led:LED_PLCC4_3.5x3.5_CCW, symbol SK6812_MINI
- added U?: NRF24L01, symbol NRF24L01
- added U?: ATMEGA328P-AU, TQFP32, symbol ATMEGA328P-AU
Connections:
- net labels added: +3.3V, LEDDRV
- net labels removed: +5C, CHARGE, PWR_EN
- wire segments 133 -> 179
